File: HUJI-Lib PCB/HUJI-Lib PCB.kicad_sch (KiCad schematic)
At the start: 11 parts

Commit message: Updated PCB files.
Parts:
- added J0: Barrel_Jack, symbol Connector:Barrel_Jack
- renumbered D-L to D-L1, D-R to D-R1
Connections:
- net at D-R1. (VIN): now also A0.12 (D12)
- net at D-L1. (VIN): now also A0.13 (D13)
- new net: A0. (VP), D-L1. (VIN), D-R1. (VIN) (x2)
Changed lines of the file:
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@@
     (comment 1 "Designed by Ido Nir and Noam Peled")
   )
+  (junction (at 128.27 93.98) (diameter 0) (color 0 0 0 0)
+  )
   (junction (at 203.2 76.2) (diameter 0) (color 0 0 0 0)
   )
+  (junction (at 132.08 81.28) (diameter 0) (color 0 0 0 0)
+  )
   (junction (at 203.2 66.04) (diameter 0) (color 0 0 0 0)
   )
   (junction (at 203.2 71.12) (diameter 0) (color 0 0 0 0)
   )
+  (wire (pts (xy 143.51 88.9) (xy 130.81 88.9))
+    (stroke (width 0) (type default) (color 0 0 0 0))
+  )
+  (wire (pts (xy 130.81 99.06) (xy 96.52 99.06))
+    (stroke (width 0) (type default) (color 0 0 0 0))
+  )
+  (wire (pts (xy 130.81 72.39) (xy 96.52 72.39))
+    (stroke (width 0) (type default) (color 0 0 0 0))
+  )
+  (wire (pts (xy 110.49 67.31) (xy 128.27 67.31))
+    (stroke (width 0) (type default) (color 0 0 0 0))
+  )
   (wire (pts (xy 186.69 71.12) (xy 190.5 71.12))
     (stroke (width 0) (type default) (color 0 0 0 0))
@@
     (stroke (width 0) (type default) (color 0 0 0 0))
   )
+  (wire (pts (xy 110.49 54.61) (xy 132.08 54.61))
+    (stroke (width 0) (type default) (color 0 0 0 0))
+  )
+  (wire (pts (xy 132.08 96.52) (xy 143.51 96.52))
+    (stroke (width 0) (type default) (color 0 0 0 0))
+  )
+  (wire (pts (xy 110.49 81.28) (xy 132.08 81.28))
+    (stroke (width 0) (type default) (color 0 0 0 0))
+  )
   (wire (pts (xy 165.1 63.5) (xy 179.07 63.5))
     (stroke (width 0) (type default) (color 0 0 0 0))
   )
+  (wire (pts (xy 110.49 93.98) (xy 128.27 93.98))
+    (stroke (width 0) (type default) (color 0 0 0 0))
+  )
   (wire (pts (xy 165.1 60.96) (xy 179.07 60.96))
     (stroke (width 0) (type default) (color 0 0 0 0))
@@
     (stroke (width 0) (type default) (color 0 0 0 0))
   )
+  (wire (pts (xy 96.52 99.06) (xy 96.52 93.98))
+    (stroke (width 0) (type default) (color 0 0 0 0))
+  )
+  (wire (pts (xy 128.27 93.98) (xy 143.51 93.98))
+    (stroke (width 0) (type default) (color 0 0 0 0))
+  )
   (wire (pts (xy 203.2 66.04) (xy 203.2 71.12))
     (stroke (width 0) (type default) (color 0 0 0 0))
   )
+  (wire (pts (xy 130.81 91.44) (xy 130.81 99.06))
+    (stroke (width 0) (type default) (color 0 0 0 0))
+  )
+  (wire (pts (xy 132.08 54.61) (xy 132.08 81.28))
+    (stroke (width 0) (type default) (color 0 0 0 0))
+  )
   (wire (pts (xy 198.12 76.2) (xy 203.2 76.2))
     (stroke (width 0) (type default) (color 0 0 0 0))
   )
+  (wire (pts (xy 132.08 81.28) (xy 132.08 96.52))
+    (stroke (width 0) (type default) (color 0 0 0 0))
+  )
+  (wire (pts (xy 96.52 67.31) (xy 96.52 72.39))
+    (stroke (width 0) (type default) (color 0 0 0 0))
+  )
   (wire (pts (xy 186.69 66.04) (xy 190.5 66.04))
     (stroke (width 0) (type default) (color 0 0 0 0))
@@
     (stroke (width 0) (type default) (color 0 0 0 0))
   )
+  (wire (pts (xy 143.51 91.44) (xy 130.81 91.44))
+    (stroke (width 0) (type default) (color 0 0 0 0))
+  )
   (wire (pts (xy 198.12 60.96) (xy 203.2 60.96))
     (stroke (width 0) (type default) (color 0 0 0 0))
@@
   )
   (wire (pts (xy 165.1 71.12) (xy 179.07 71.12))
+    (stroke (width 0) (type default) (color 0 0 0 0))
+  )
+  (wire (pts (xy 130.81 88.9) (xy 130.81 72.39))
+    (stroke (width 0) (type default) (color 0 0 0 0))
+  )
+  (wire (pts (xy 128.27 67.31) (xy 128.27 93.98))
     (stroke (width 0) (type default) (color 0 0 0 0))
   )
@@
   (symbol (lib_id "Component Library:PE-IR Sensor") (at 101.6 68.58 0) (unit 1)
     (in_bom yes) (on_board yes) (fields_autoplaced)
-    (property "Reference" "D-R" (id 0) (at 114.3 60.3249 0)
+    (property "Reference" "D-R1" (id 0) (at 114.3 60.3249 0)
       (effects (font (size 1.27 1.27)) (justify left))
     )
@@
     (pin "")
     (pin "")
+  )
+  (symbol (lib_id "Connector:Barrel_Jack") (at 123.19 109.22 0) (unit 1)
+    (in_bom yes) (on_board yes) (fields_autoplaced)
+    (property "Reference" "J0" (id 0) (at 123.19 100.33 0))
+    (property "Value" "Barrel_Jack" (id 1) (at 123.19 102.87 0))
+    (property "Footprint" "" (id 2) (at 124.46 110.236 0)
+      (effects (font (size 1.27 1.27)) hide)
+    )
+    (property "Datasheet" "~" (id 3) (at 124.46 110.236 0)
+      (effects (font (size 1.27 1.27)) hide)
+    )
+    (pin "1")
+    (pin "2")
   )
   (symbol (lib_id "Device:R") (at 182.88 66.04 90) (unit 1)
@@
   (symbol (lib_id "Component Library:PE-IR Sensor") (at 101.6 95.25 0) (unit 1)
     (in_bom yes) (on_board yes) (fields_autoplaced)
-    (property "Reference" "D-L" (id 0) (at 114.3 86.9949 0)
+    (property "Reference" "D-L1" (id 0) (at 114.3 86.9949 0)
       (effects (font (size 1.27 1.27)) (justify left))
     )
@@
     )
     (path "/ee754bbf-9028-488e-b236-c1e77ca5d275"
-      (reference "D-L") (unit 1) (value "PE-IR Sensor") (footprint "")
+      (reference "D-L1") (unit 1) (value "PE-IR Sensor") (footprint "")
     )
     (path "/b31d0e33-93c1-4260-a1eb-23c2d0216b92"
-      (reference "D-R") (unit 1) (value "PE-IR Sensor") (footprint "")
+      (reference "D-R1") (unit 1) (value "PE-IR Sensor") (footprint "")
     )
     (path "/10adf1cc-2eb7-4164-b74a-66a84a32f9fc"
@@
       (reference "D4") (unit 1) (value "LED") (footprint "")
     )
+    (path "/be68608f-ef59-4ecb-8c54-5775ee858935"
+      (reference "J0") (unit 1) (value "Barrel_Jack") (footprint "")
+    )
     (path "/2c6dc056-fea6-4c97-85ce-c64978655430"
